Commit message: Sensor position corrected

File: racecar/model/racecar.xacro (robot description, xacro)
@@ -1,107 +1,218 @@
 <?xml version="1.0"?>
-<!-- A simple model of the racecar for rviz -->
-<robot xmlns:xacro="http://www.ros.org/wiki/xacro" name="racecar">
-  <xacro:property name="wheelbase" value="0.325" />
-  <xacro:property name="width" value="0.2" />
-  <xacro:property name="height" value="0.1" />
-  <xacro:property name="ground_offset" value="0.04" />
-  <xacro:property name="wheel_radius" value="0.05" />
-  <xacro:property name="wheel_length" value="0.045" />
-  <xacro:property name="laser_distance_from_base_link" value="0.275" />
-  <xacro:property name="laser_height" value="0.05" />
-  <xacro:property name="laser_radius" value="0.026" />
-  <material name="black">
-    <color rgba="0.2 0.2 0.2 1."/>
-  </material>
-  <material name="blue">
-    <color rgba="0.3 0.57 1. 1."/>
-  </material>
-  <link name="base_link">
-    <visual>
-      <origin xyz="${wheelbase/2} 0 ${ground_offset+height/2}"/>
+<robot name="racecar" xmlns:xacro="http://www.ros.org/wiki/xacro">
+  <xacro:include filename="$(find racecar_description)/urdf/macros.xacro" />
+  <!-- Add chassis and it's inertia link -->
+  <link name="base_link" />
+  <link name="chassis">
+    <visual>
+      <xacro:chassis_geometry/>
+      <material name="green" />
+    </visual>
+  </link>
+  <joint name="base_link_joint" type="fixed">
+    <origin xyz="0 0 0.05" rpy="0 0 0" />
+    <parent link="base_link" />
+    <child link="chassis" />
+  </joint>
+  <link name="chassis_inertia">
+    <inertial>
+      <xacro:chassis_inertial_params />
+    </inertial>
+  </link>
+  <joint name="chassis_inertia_joint" type="fixed">
+    <origin xyz="0 0 0" rpy="0 0 0" />
+    <parent link="chassis" />
+    <child link="chassis_inertia" />
+  </joint>
+  <!-- Add the left rear wheel with its joints and tranmissions -->
+  <link name="left_rear_wheel">
+    <inertial>
+      <xacro:left_wheels_inertial_params />
+    </inertial>
+    <visual>
+      <xacro:left_rear_wheel_geometry />
+      <material name="black" />
+    </visual>
+    <collision>robot
+      <xacro:left_wheels_collision_geometry />
+    </collision>
+  </link>
+  <joint name="left_rear_wheel_joint" type="continuous">
+    <origin xyz="0 0.1 0" rpy="1.5708 0 0" />
+    <parent link="chassis" />
+    <child link="left_rear_wheel" />
+    <axis xyz="0 0 -1" />
+    <limit effort="10" velocity="100" />
+  </joint>
+  <xacro:wheel_transmission name="left_rear_wheel" />
+  <!-- Add the right rear wheel with its joints and tranmissions -->
+  <link name="right_rear_wheel">
+    <inertial>
+      <xacro:right_wheels_inertial_params />
+    </inertial>
+    <visual>
+      <xacro:right_rear_wheel_geometry />
+      <material name="black" />
+    </visual>
+    <collision>
+      <xacro:right_wheels_collision_geometry />
+    </collision>
+  </link>
+  <joint name="right_rear_wheel_joint" type="continuous">
+    <origin xyz="0 -0.1 0" rpy="1.5708 0 0" />
+    <parent link="chassis" />
+    <child link="right_rear_wheel" />
+    <axis xyz="0 0 -1" />
+    <limit effort="10" velocity="100" />
+  </joint>
+  <xacro:wheel_transmission name="right_rear_wheel" />
+  <!-- Add the left steering hinge with its joints and tranmissions -->
+  <link name="left_steering_hinge">
+    <inertial>
+      <xacro:steering_hinge_inertial_params />
+    </inertial>
+    <visual>
+      <xacro:left_steering_hinge_geometry />
+      <material name="grey" />
+    </visual>
+  </link>
+  <joint name="left_steering_hinge_joint" type="revolute">
+    <origin xyz="0.325 0.1 0" rpy="0 1.5708 0" />
+    <parent link="chassis" />
+    <child link="left_steering_hinge" />
+    <axis xyz="-1 0 0" />
+    <limit lower="-1.0" upper="1.0" effort="10" velocity="100" />
+  </joint>
+  <xacro:steering_hinge_transmission name="left_steering_hinge" />
+  <!-- Add the right steering hinge with its joints and tranmissions -->
+  <link name="right_steering_hinge">
+    <inertial>
+      <xacro:steering_hinge_inertial_params />
+    </inertial>
+    <visual>
+      <xacro:right_steering_hinge_geometry />
+      <material name="grey" />
+    </visual>
+  </link>
+  <joint name="right_steering_hinge_joint" type="continuous">
+    <origin xyz="0.325 -0.1 0" rpy="0 1.5708 0" />
+    <parent link="chassis" />
+    <child link="right_steering_hinge" />
+    <axis xyz="-1 0 0" />
+    <limit lower="-1.0" upper="1.0" effort="10" velocity="100" />
+  </joint>
+  <xacro:steering_hinge_transmission name="right_steering_hinge" />
+  <!-- Add the left front wheel with its joints and tranmissions -->
+  <link name="left_front_wheel">
+    <inertial>
+      <xacro:left_wheels_inertial_params />
+    </inertial>
+    <visual>
+      <xacro:left_front_wheel_geometry />
+      <material name="black" />
+    </visual>
+    <collision>
+      <xacro:left_wheels_collision_geometry />
+    </collision>
+  </link>
+  <joint name="left_front_wheel_joint" type="continuous">
+    <origin xyz="0 0 0" rpy="1.5708 0 0" />
+    <parent link="left_steering_hinge" />
+    <child link="left_front_wheel" />
+    <axis xyz="0 0 -1" />
+    <limit effort="10" velocity="100" />
+  </joint>
+  <xacro:wheel_transmission name="left_front_wheel" />
+  <!-- Add the left front wheel with its joints and tranmissions -->
+  <link name="right_front_wheel">
+    <inertial>
+      <xacro:right_wheels_inertial_params />
+    </inertial>
+    <visual>
+      <xacro:right_front_wheel_geometry />
+      <material name="black" />
+    </visual>
+    <collision>
+      <xacro:right_wheels_collision_geometry />
+    </collision>
+  </link>
+  <joint name="right_front_wheel_joint" type="continuous">
+    <origin xyz="0 0 0" rpy="1.5708 0 0" />
+    <parent link="right_steering_hinge" />
+    <child link="right_front_wheel" />
+    <axis xyz="0 0 -1" />
+    <limit effort="10" velocity="100"/>
+  </joint>
+  <xacro:wheel_transmission name="right_front_wheel" />
+  <!-- Add Hokuyo laser scanner -->
+  <link name="laser">
+    <inertial>
+      <xacro:hokuyo_inertial_params />
+    </inertial>
+    <collision>
+      <origin xyz="0 0 0" rpy="0 0 0"/>
       <geometry>
-        <box size="${wheelbase} ${width} ${height}"/>
+        <box size="0.1 0.1 0.1"/>
       </geometry>
-      <material name="blue"/>
-    </visual>
-  </link>
-  <joint name="base_to_laser_model" type="fixed">
-    <parent link="base_link"/>
-    <child link="laser_model"/>
-    <origin xyz="${laser_distance_from_base_link} 0 ${ground_offset+height+(laser_height/2)}"/>
-  </joint>
-  <link name="laser_model">
-    <visual>
+    </collision>
+    <visual>
+      <origin xyz="0 0 0" rpy="0 0 0"/>
       <geometry>
-        <cylinder radius="${laser_radius}" length="${laser_height}"/>
+        <mesh filename="package://racecar_description/meshes/hokuyo.dae"/>
+        <material name="grey" />
       </geometry>
-      <material name="black"/>
-    </visual>
-  </link>
-  <joint name="base_to_back_left_wheel" type="fixed">
-    <parent link="base_link"/>
-    <child link="back_left_wheel"/>
-    <origin xyz="0 ${(wheel_length+width)/2} ${wheel_radius}"/>
-  </joint>
-  <link name="back_left_wheel">
-    <visual>
+    </visual>
+  </link>
+  <joint name="hokuyo_joint" type="fixed">
+    <origin xyz="0.285 0.0 0.24" rpy="0 0 0"/>
+    <parent link="chassis" />
+    <child link="laser" />
+    <axis xyz="0 0 1" />
+  </joint>
+  <!-- NVIDIA Xavier -->
+  <!-- Original StereoLabs ZED Camera URDF file -->
+  <link name="zed_camera_center">
+    <visual>
+      <origin xyz="0 0 0" rpy="0 0 0"/>
       <geometry>
-        <cylinder radius="${wheel_radius}" length="${wheel_length}"/>
+          <mesh filename="package://zed_wrapper/urdf/models/ZED.stl" />
       </geometry>
-      <material name="black"/>
-      <origin rpy="${pi/2} 0 0"/>
-    </visual>
-  </link>
-  <joint name="base_to_back_right_wheel" type="fixed">
-    <parent link="base_link"/>
-    <child link="back_right_wheel"/>
-    <origin xyz="0 ${-(wheel_length+width)/2} ${wheel_radius}"/>
-  </joint>
-  <link name="back_right_wheel">
-    <visual>
-      <geometry>
-        <cylinder radius="${wheel_radius}" length="${wheel_length}"/>
-      </geometry>
-      <material name="black"/>
-      <origin rpy="${pi/2} 0 0"/>
-    </visual>
-  </link>
-  <joint name="base_to_front_left_hinge" type="fixed">
-    <parent link="base_link"/>
-    <child link="front_left_hinge"/>
-    <origin xyz="${wheelbase} ${(wheel_length+width)/2} ${wheel_radius}"/>
-  </joint>
-  <link name="front_left_hinge"/>
-  <joint name="front_left_hinge_to_wheel" type="continuous">
-    <parent link="front_left_hinge"/>
-    <child link="front_left_wheel"/>
-  </joint>
-  <link name="front_left_wheel">
-    <visual>
-      <geometry>
-        <cylinder radius="${wheel_radius}" length="${wheel_length}"/>
-      </geometry>
-      <material name="black"/>
-      <origin rpy="${pi/2} 0 0"/>
-    </visual>
-  </link>
-  <joint name="base_to_front_right_hinge" type="fixed">
-    <parent link="base_link"/>
-    <child link="front_right_hinge"/>
-    <origin xyz="${wheelbase} ${-(wheel_length+width)/2} ${wheel_radius}"/>
-  </joint>
-  <link name="front_right_hinge"/>
-  <joint name="front_right_hinge_to_wheel" type="continuous">
-    <parent link="front_right_hinge"/>
-    <child link="front_right_wheel"/>
-  </joint>
-  <link name="front_right_wheel">
-    <visual>
-      <geometry>
-        <cylinder radius="${wheel_radius}" length="${wheel_length}"/>
-      </geometry>
-      <material name="black"/>
-      <origin rpy="${pi/2} 0 0"/>
-    </visual>
-  </link>
+      <material name="light_grey" />
+    </visual>
+  </link>
+  <joint name="zed_camera_joint" type="fixed">
+    <origin xyz="0.340 0 0.24" rpy="0 0 0"/>
+    <parent link="chassis"/>
+    <child link="zed_camera_center"/>
+    <axis xyz="0 0 1" />
+    <!-- <limit lower="0.0" upper="0.0" effort="0.0" velocity="0.0" /> -->
+  </joint>
+<!-- Left Camera -->
+    <joint name="zed_left_camera_joint" type="fixed">
+        <parent link="zed_camera_center"/>
+        <child link="zed_left_camera_frame"/>
+        <origin xyz="0 0.06 0" rpy="0 0 0" />
+    </joint>
+    <link name="zed_left_camera_frame" />
+    <joint name="zed_left_camera_optical_joint" type="fixed">
+        <origin xyz="0 0 0" rpy="-1.57079632679 0.0 -1.57079632679"/>
+        <parent link="zed_left_camera_frame"/>
+        <child link="zed_left_camera_optical_frame"/>
+    </joint>
+    <link name="zed_left_camera_optical_frame"/>
+<!-- Right Camera -->
+    <joint name="zed_right_camera_joint" type="fixed">
+        <parent link="zed_camera_center"/>
+        <child link="zed_right_camera_frame"/>
+        <origin xyz="0 -0.06 0" rpy="0 0 0" />
+    </joint>
+    <link name="zed_right_camera_frame" />
+    <joint name="zed_right_camera_optical_joint" type="fixed">
+        <origin xyz="0 0 0" rpy="-1.57079632679 0.0 -1.57079632679"/>
+        <parent link="zed_right_camera_frame"/>
+        <child link="zed_right_camera_optical_frame"/>
+    </joint>
+    <link name="zed_right_camera_optical_frame"/>
+  <!-- Add the remaining xacros -->
+  <xacro:include filename="$(find racecar_description)/urdf/materials.xacro" />
 </robot>
